Commit message: Show the workcell in 3D and load URDF meshes from robots/
- The web serves robots/ at /robots/ (nginx read-only mount in compose; a
  Vite plugin in dev with path-escape and missing-file 404s), so URDF
  package:// meshes and workcell files load in the browser
- robot.yaml gains mesh_packages (package -> folder, default = package
  name) and scene objects (box / cylinder / sphere / STL-GLB mesh, xyz and
  rpy relative to the robot base); the executor publishes /robot_scene
- Viewer: workcell drawn with the robot and in the twin, grid lowered to
  the lowest object (no z-fighting with the bench top), URDF built once
  the mesh locations are known, GLB support, ghost tint for late meshes,
  a notice when a 3D file fails to load
- Demo: base_link uses an STL via package://, plus a bench, jig, part and
  box matching the mock camera scene
- scene3d.test.js (coordinates, rpy order, cylinder axis, mesh URLs) in CI;
  smoke test checks /robot_scene

Co-Authored-By: Claude Opus 5.5 <noreply@anthropic.com>

File: robots/demo_arm/robot.urdf (robot description, URDF)
Before this commit: robot demo_arm, 7 links, 6 joints
Links:
- link base_link: geometry visual mesh filename=package://demo_arm/meshes/base.stl

Commit message: Let the profile pick the tool tip for the path preview; fit the example to the work cell
robot.yaml tcp_link names the URDF link whose path the 3D preview draws
(falls back to the deepest leaf link, warns in the 3D view if missing).
The demo URDF gets a fixed tool_tip link at the finger tips. The example
pick-and-place joint values now put the tool tip, pointing down, over the
demo part and box, with a descend-to-pick and lift step.

Co-Authored-By: Claude Opus 5.5 <noreply@anthropic.com>

File: robots/demo_arm/robot.urdf (robot description, URDF)
Before this commit: robot demo_arm, 7 links, 6 joints
Links:
- added link tool_tip
Joints:
- added joint tool_tip_joint: type fixed, parent link6, child tool_tip, origin xyz=0 0 0.11
